File: PCB/MYHACKPAD.kicad_pcb (KiCad board)
At the start: 2 copper layers, 65.1 x 65.1 mm, 15 parts, among them J1 OLED_128x32, SW1 SW_Push, SW2 SW_Push, SW3 SW_Push, SW4 SW_Push, SW5 SW_Push, SW6 RotaryEncoder_Switch, U1 XIAO-RP2040-DIP

Commit message: update readme + kicad
Parts:
- D1: footprint LED_SMD:LED_SK6812MINI_PLCC4_3.5x3.5mm_P1.75mm -> SK6812 Mini-E:SK6812MINI-E_fixed
Routing:
- net GND: track 81.0 -> 69.9 mm
- net VCC: track 87.8 -> 96.8 mm, vias 3 -> 6
- net SK6812MINI: track 52.6 -> 51.7 mm, vias 1 -> 0
- added copper zone on B.Cu, net GND
- added copper zone on F.Cu, net GND
