File: PCB/MYHACKPAD.kicad_sch (KiCad schematic)
At the start: 15 parts, among them J1 OLED_128x32, SW1 SW_Push, SW2 SW_Push, SW3 SW_Push, SW4 SW_Push, SW5 SW_Push, SW6 RotaryEncoder_Switch, U1 XIAO-RP2040-DIP

Commit message: update readme + kicad
Parts:
- D1: footprint LED_SMD:LED_SK6812MINI_PLCC4_3.5x3.5mm_P1.75mm -> SK6812 Mini-E:SK6812MINI-E_fixed
Connections:
- no-connect marks 0 -> 1
Changed lines of the file:
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@@
 		(color 0 0 0 0)
+	)
+	(no_connect
+		(at 68.58 166.37)
 	)
 	(wire
@@
 			)
 		)
-		(property "Footprint" "LED_SMD:LED_SK6812MINI_PLCC4_3.5x3.5mm_P1.75mm"
+		(property "Footprint" "SK6812 Mini-E:SK6812MINI-E_fixed"
 			(at 62.23 173.99 0)
 			(effects
